File: hardware/pdsupply-PPS/pdsupply-PPS.kicad_sch (KiCad schematic)
At the start: 74 parts, among them IC1 LTM8083EY#PBF, IC2 FPF2895UCX, J1 USB4505-03-0-A_REVA, J2 USB4505-03-0-A_REVA, J3 Screw_Terminal_01x02, U1 FUSB307BMPX, U2 ADUM3160, U3 ACS71240KEXBLT-050U5, U4 STM32L432KCUx

Commit message: component placement done
Connections:
- net +3V3: now also U2.1 (VBUS1), U2.3 (VDD1), U2.5 (SPU); no longer U2.12 (PIN), U2.13 (SPD), U2.14 (VDD2), U2.16 (VBUS2)
- net +5V: now also U2.16 (VBUS2); no longer U2.1 (VBUS1)
- net GND: now also J3.2 (Pin_2), U2.2 (GND1), U2.8 (GND1); no longer J3.1 (Pin_1), U2.15 (GND2), U2.9 (GND2)
- net GND1: now also U2.15 (GND2), U2.9 (GND2); no longer U2.2 (GND1), U2.8 (GND1)
- net USB_DM: now also U2.6 (UD-); no longer U2.11 (DD-)
- net USB_DP: now also U2.7 (UD+); no longer U2.10 (DD+)
- net at JP1.1 (A), R11.2: now also U2.10 (DD+); no longer U2.7 (UD+)
- net at U3.3 (IP-): now also J3.1 (Pin_1); no longer J3.2 (Pin_2)
- net at JP2.1 (A), R12.1: now also U2.11 (DD-); no longer U2.6 (UD-)
- new net: C11.1, U2.13 (SPD), U2.14 (VDD2)
- now unconnected: U2.4 (PDEN)
Other:
- moved on the sheet: J3
Changed lines of the file:
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@@
-    (stroke (width 0) (type default) (color 0 0 0 0))
-  )
-  (wire (pts (xy 303.53 91.44) (xy 303.53 97.79))
     (stroke (width 0) (type default) (color 0 0 0 0))
   )
@@
     (stroke (width 0) (type default) (color 0 0 0 0))
   )
+  (wire (pts (xy 298.45 89.535) (xy 298.45 97.79))
+    (stroke (width 0) (type default) (color 0 0 0 0))
+  )
   (wire (pts (xy 387.985 170.18) (xy 400.05 170.18))
     (stroke (width 0) (type default) (color 0 0 0 0))
@@
     (stroke (width 0) (type default) (color 0 0 0 0))
   )
-  (wire (pts (xy 303.53 97.79) (xy 321.945 97.79))
+  (wire (pts (xy 298.45 97.79) (xy 321.945 97.79))
     (stroke (width 0) (type default) (color 0 0 0 0))
   )
@@
     (stroke (width 0) (type default) (color 0 0 0 0))
   )
+  (wire (pts (xy 296.545 86.995) (xy 298.45 86.995))
+    (stroke (width 0) (type default) (color 0 0 0 0))
+  )
   (wire (pts (xy 270.51 254) (xy 271.78 254))
     (stroke (width 0) (type default) (color 0 0 0 0))
@@
     (stroke (width 0) (type default) (color 0 0 0 0))
   )
-  (wire (pts (xy 296.545 88.9) (xy 296.545 76.835))
+  (wire (pts (xy 296.545 76.835) (xy 296.545 86.995))
     (stroke (width 0) (type default) (color 0 0 0 0))
   )
@@
     (stroke (width 0) (type default) (color 0 0 0 0))
   )
-  (wire (pts (xy 289.56 88.9) (xy 296.545 88.9))
-    (stroke (width 0) (type default) (color 0 0 0 0))
-  )
   (wire (pts (xy 88.9 140.335) (xy 88.9 135.89))
     (stroke (width 0) (type default) (color 0 0 0 0))
@@
   )
   (wire (pts (xy 68.58 66.04) (xy 68.58 79.375))
-    (stroke (width 0) (type default) (color 0 0 0 0))
-  )
-  (wire (pts (xy 289.56 91.44) (xy 303.53 91.44))
     (stroke (width 0) (type default) (color 0 0 0 0))
   )
@@
     (pin "2")
   )
-  (symbol (lib_id "Interface_USB:ADUM3160") (at 266.7 228.6 0) (unit 1)
-    (in_bom yes) (on_board yes)
-    (property "Reference" "U2" (id 0) (at 256.54 214.63 0)
-      (effects (font (size 1.27 1.27)) (justify left))
-    )
-    (property "Value" "ADUM3160" (id 1) (at 270.51 214.63 0)
+  (symbol (lib_id "Interface_USB:ADUM3160") (at 266.7 228.6 0) (mirror y) (unit 1)
+    (in_bom yes) (on_board yes)
+    (property "Reference" "U2" (id 0) (at 276.86 214.63 0)
+      (effects (font (size 1.27 1.27)) (justify left))
+    )
+    (property "Value" "ADUM3160" (id 1) (at 262.89 214.63 0)
       (effects (font (size 1.27 1.27)) (justify left))
     )
@@
       (effects (font (size 1.27 1.27)) hide)
     )
-    (property "Datasheet" "https://www.analog.com/media/en/technical-documentation/data-sheets/ADuM3160.pdf" (id 3) (at 261.62 228.6 0)
+    (property "Datasheet" "https://www.analog.com/media/en/technical-documentation/data-sheets/ADuM3160.pdf" (id 3) (at 271.78 228.6 0)
       (effects (font (size 1.27 1.27)) hide)
     )
@@
     (pin "1")
   )
-  (symbol (lib_id "Connector:Screw_Terminal_01x02") (at 284.48 91.44 180) (unit 1)
-    (in_bom yes) (on_board yes) (fields_autoplaced)
-    (property "Reference" "J3" (id 0) (at 284.48 82.55 0))
-    (property "Value" "Screw_Terminal_01x02" (id 1) (at 284.48 85.09 0))
-    (property "Footprint" "TerminalBlock_Phoenix:TerminalBlock_Phoenix_MKDS-1,5-2_1x02_P5.00mm_Horizontal" (id 2) (at 284.48 91.44 0)
-      (effects (font (size 1.27 1.27)) hide)
-    )
-    (property "Datasheet" "~" (id 3) (at 284.48 91.44 0)
-      (effects (font (size 1.27 1.27)) hide)
-    )
+  (symbol (lib_id "Connector:Screw_Terminal_01x02") (at 303.53 86.995 0) (unit 1)
+    (in_bom yes) (on_board yes)
+    (property "Reference" "J3" (id 0) (at 306.07 86.9949 0)
+      (effects (font (size 1.27 1.27)) (justify left))
+    )
+    (property "Value" "Screw_Terminal_01x02" (id 1) (at 302.26 92.71 0)
+      (effects (font (size 1.27 1.27)) (justify left))
+    )
+    (property "Footprint" "TerminalBlock_Phoenix:TerminalBlock_Phoenix_MKDS-1,5-2_1x02_P5.00mm_Horizontal" (id 2) (at 303.53 86.995 0)
+      (effects (font (size 1.27 1.27)) hide)
+    )
+    (property "Datasheet" "~" (id 3) (at 303.53 86.995 0)
+      (effects (font (size 1.27 1.27)) hide)
+    )

Commit message: added few routes
Connections:
- net +3V3: now also U2.12 (PIN), U2.13 (SPD), U2.14 (VDD2), U2.16 (VBUS2); no longer U2.1 (VBUS1), U2.3 (VDD1), U2.5 (SPU)
- net +5V: now also U2.1 (VBUS1); no longer U2.16 (VBUS2)
- net GND: now also U2.15 (GND2), U2.9 (GND2); no longer U2.2 (GND1), U2.8 (GND1)
- net GND1: now also U2.2 (GND1), U2.8 (GND1); no longer U2.15 (GND2), U2.9 (GND2)
- net USB_DM: now also U2.11 (DD-); no longer U2.6 (UD-)
- net USB_DP: now also U2.10 (DD+); no longer U2.7 (UD+)
- net at JP1.1 (A), R11.2: now also U2.7 (UD+); no longer U2.10 (DD+)
- net Vbus_pre: now reaches C13.1, IC2.C2 (VOUT_1), IC2.D1 (VOUT_2), IC2.D2 (VOUT_3), IC2.E1 (VOUT_4), IC2.E2 (VOUT_5), IC2.F1 (VOUT_6), IC2.F2 (VOUT_7), U3.1 (IP+)
- net VBus_Out: now reaches J3.1 (Pin_1), U3.3 (IP-)
- net at JP2.1 (A), R12.1: now also U2.6 (UD-); no longer U2.11 (DD-)
- net at U2.4 (PDEN): now also C11.1, U2.3 (VDD1), U2.5 (SPU)

Commit message: almost done with routing
Connections:
- net +3.3V_Pre: now reaches C8.1, FB3.1, IC1.F3 (ISN), IC1.F4 (VOUT_1), IC1.F5 (VOUT_2), IC1.G3 (ISP), IC1.G4 (VOUT_3), IC1.G5 (VOUT_4), R8.1
Changed lines of the file:
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@@
+    (effects (font (size 1.27 1.27)) (justify left bottom))
+  )
+  (label "+3.3V_Pre" (at 164.465 139.7 0)
     (effects (font (size 1.27 1.27)) (justify left bottom))
   )
@@
     (pin "1")
   )
-  (symbol (lib_id "Device:R_Small_US") (at 105.41 185.42 0) (unit 1)
-    (in_bom yes) (on_board yes)
-    (property "Reference" "R3" (id 0) (at 101.6 185.42 0)
-      (effects (font (size 1.27 1.27)) (justify left))
-    )
-    (property "Value" "40.2k" (id 1) (at 107.315 185.42 0)
-      (effects (font (size 1.27 1.27)) (justify left))
-    )
+  (symbol (lib_id "Device:R_Small_US") (at 105.41 185.42 0) (mirror y) (unit 1)
+    (in_bom yes) (on_board yes)
+    (property "Reference" "R3" (id 0) (at 109.22 185.42 0)
+      (effects (font (size 1.27 1.27)) (justify left))
+    )
+    (property "Value" "40.2k" (id 1) (at 103.505 185.42 0)
+      (effects (font (size 1.27 1.27)) (justify left))
+    )

Commit message: almost done
Parts:
- added H1, H2, H3, H4: MountingHole_Pad, MountingHole:MountingHole_3mm, symbol Mechanical:MountingHole_Pad
Connections:
- net GND: now also H1.1, H2.1, H3.1, H4.1
Changed lines of the file:
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@@
   (junction (at 226.695 256.54) (diameter 0) (color 0 0 0 0)
   )
+  (junction (at 31.75 202.565) (diameter 0) (color 0 0 0 0)
+  )
   (junction (at 109.855 139.7) (diameter 0) (color 0 0 0 0)
   )
   (junction (at 134.62 35.56) (diameter 0) (color 0 0 0 0)
   )
+  (junction (at 31.75 191.135) (diameter 0) (color 0 0 0 0)
+  )
   (junction (at 68.58 79.375) (diameter 0) (color 0 0 0 0)
   )
@@
   (junction (at 326.39 126.365) (diameter 0) (color 0 0 0 0)
   )
+  (junction (at 31.75 216.535) (diameter 0) (color 0 0 0 0)
+  )
   (junction (at 365.76 182.88) (diameter 0) (color 0 0 0 0)
   )
@@
     (stroke (width 0) (type default) (color 0 0 0 0))
   )
+  (wire (pts (xy 27.305 216.535) (xy 31.75 216.535))
+    (stroke (width 0) (type default) (color 0 0 0 0))
+  )
   (wire (pts (xy 112.395 175.26) (xy 105.41 175.26))
     (stroke (width 0) (type default) (color 0 0 0 0))
@@
     (stroke (width 0) (type default) (color 0 0 0 0))
   )
+  (wire (pts (xy 31.75 216.535) (xy 31.75 220.98))
+    (stroke (width 0) (type default) (color 0 0 0 0))
+  )
   (wire (pts (xy 321.945 165.1) (xy 329.565 165.1))
     (stroke (width 0) (type default) (color 0 0 0 0))
@@
     (stroke (width 0) (type default) (color 0 0 0 0))
   )
+  (wire (pts (xy 27.305 191.135) (xy 31.75 191.135))
+    (stroke (width 0) (type default) (color 0 0 0 0))
+  )
   (wire (pts (xy 360.68 197.485) (xy 360.68 199.39))
     (stroke (width 0) (type default) (color 0 0 0 0))
@@
     (stroke (width 0) (type default) (color 0 0 0 0))
   )
+  (wire (pts (xy 31.75 179.07) (xy 31.75 191.135))
+    (stroke (width 0) (type default) (color 0 0 0 0))
+  )
   (wire (pts (xy 57.785 130.81) (xy 59.69 130.81))
     (stroke (width 0) (type default) (color 0 0 0 0))
@@
     (stroke (width 0) (type default) (color 0 0 0 0))
   )
+  (wire (pts (xy 27.305 179.07) (xy 31.75 179.07))
+    (stroke (width 0) (type default) (color 0 0 0 0))
+  )
   (wire (pts (xy 96.52 149.86) (xy 96.52 151.765))
     (stroke (width 0) (type default) (color 0 0 0 0))
   )
+  (wire (pts (xy 31.75 202.565) (xy 31.75 216.535))
+    (stroke (width 0) (type default) (color 0 0 0 0))
+  )
   (wire (pts (xy 156.845 238.125) (xy 156.845 240.665))
     (stroke (width 0) (type default) (color 0 0 0 0))
@@
     (stroke (width 0) (type default) (color 0 0 0 0))
   )
+  (wire (pts (xy 27.305 202.565) (xy 31.75 202.565))
+    (stroke (width 0) (type default) (color 0 0 0 0))
+  )
   (wire (pts (xy 38.735 127) (xy 38.735 130.81))
     (stroke (width 0) (type default) (color 0 0 0 0))
@@
     (stroke (width 0) (type default) (color 0 0 0 0))
   )
+  (wire (pts (xy 31.75 191.135) (xy 31.75 202.565))
+    (stroke (width 0) (type default) (color 0 0 0 0))
+  )
   (wire (pts (xy 207.645 226.06) (xy 213.36 226.06))
     (stroke (width 0) (type default) (color 0 0 0 0))
@@
     (pin "9")
   )
+  (symbol (lib_id "power:GND") (at 31.75 220.98 0) (unit 1)
+    (in_bom yes) (on_board yes) (fields_autoplaced)
+    (property "Reference" "#PWR0101" (id 0) (at 31.75 227.33 0)
+      (effects (font (size 1.27 1.27)) hide)
+    )
+    (property "Value" "GND" (id 1) (at 31.75 225.425 0))
+    (property "Footprint" "" (id 2) (at 31.75 220.98 0)
+      (effects (font (size 1.27 1.27)) hide)
+    )
+    (property "Datasheet" "" (id 3) (at 31.75 220.98 0)
+      (effects (font (size 1.27 1.27)) hide)
+    )
+    (pin "1")
+  )
   (symbol (lib_id "Device:R_Small_US") (at 328.295 158.75 0) (unit 1)
     (in_bom yes) (on_board yes)
@@
     (pin "9")
   )
+  (symbol (lib_id "Mechanical:MountingHole_Pad") (at 24.765 202.565 90) (unit 1)
+    (in_bom yes) (on_board yes) (fields_autoplaced)
+    (property "Reference" "H3" (id 0) (at 23.495 195.58 90))
+    (property "Value" "MountingHole_Pad" (id 1) (at 23.495 198.12 90))
+    (property "Footprint" "MountingHole:MountingHole_3mm" (id 2) (at 24.765 202.565 0)
+      (effects (font (size 1.27 1.27)) hide)
+    )
+    (property "Datasheet" "~" (id 3) (at 24.765 202.565 0)
+      (effects (font (size 1.27 1.27)) hide)
+    )
+    (pin "1")
+  )
   (symbol (lib_id "Device:D_Schottky_Small") (at 57.785 63.5 270) (unit 1)
     (in_bom yes) (on_board yes) (fields_autoplaced)
@@
     (pin "2")
   )
+  (symbol (lib_id "Mechanical:MountingHole_Pad") (at 24.765 179.07 90) (unit 1)
+    (in_bom yes) (on_board yes) (fields_autoplaced)
+    (property "Reference" "H1" (id 0) (at 23.495 171.45 90))
+    (property "Value" "MountingHole_Pad" (id 1) (at 23.495 173.99 90))
+    (property "Footprint" "MountingHole:MountingHole_3mm" (id 2) (at 24.765 179.07 0)
+      (effects (font (size 1.27 1.27)) hide)
+    )
+    (property "Datasheet" "~" (id 3) (at 24.765 179.07 0)
+      (effects (font (size 1.27 1.27)) hide)
+    )
+    (pin "1")
+  )
   (symbol (lib_id "Device:C_Small") (at 272.415 44.45 0) (unit 1)
     (in_bom yes) (on_board yes) (fields_autoplaced)
@@
     (pin "1")
   )
+  (symbol (lib_id "Mechanical:MountingHole_Pad") (at 24.765 191.135 90) (unit 1)
+    (in_bom yes) (on_board yes) (fields_autoplaced)
+    (property "Reference" "H2" (id 0) (at 23.495 184.15 90))
+    (property "Value" "MountingHole_Pad" (id 1) (at 23.495 186.69 90))
+    (property "Footprint" "MountingHole:MountingHole_3mm" (id 2) (at 24.765 191.135 0)
+      (effects (font (size 1.27 1.27)) hide)
+    )
+    (property "Datasheet" "~" (id 3) (at 24.765 191.135 0)
+      (effects (font (size 1.27 1.27)) hide)
+    )
+    (pin "1")
+  )
   (symbol (lib_id "USB4505-03-0-A_REVA:USB4505-03-0-A_REVA") (at 170.815 227.33 0) (unit 1)
     (in_bom yes) (on_board yes)
@@
     (pin "9")
   )
+  (symbol (lib_id "Mechanical:MountingHole_Pad") (at 24.765 216.535 90) (unit 1)
+    (in_bom yes) (on_board yes) (fields_autoplaced)
+    (property "Reference" "H4" (id 0) (at 23.495 209.55 90))
+    (property "Value" "MountingHole_Pad" (id 1) (at 23.495 212.09 90))
+    (property "Footprint" "MountingHole:MountingHole_3mm" (id 2) (at 24.765 216.535 0)
+      (effects (font (size 1.27 1.27)) hide)
+    )
+    (property "Datasheet" "~" (id 3) (at 24.765 216.535 0)
+      (effects (font (size 1.27 1.27)) hide)
+    )
+    (pin "1")
+  )
   (symbol (lib_name "RCU-0C_1") (lib_id "RCU-0C:RCU-0C") (at 374.65 197.485 270) (unit 1)
     (in_bom yes) (on_board yes)
@@
       (reference "#PWR035") (unit 1) (value "+3.3V") (footprint "")
     )
+    (path "/22aa5139-3981-4f8a-84ad-deca672782ea"
+      (reference "#PWR0101") (unit 1) (value "GND") (footprint "")
+    )
     (path "/5fa9c18e-a21f-4331-abe2-b895eed2ac96"
       (reference "+3.3V1") (unit 1) (value "RCU-0C") (footprint "RCU-0C:TP+195X110")
@@
       (reference "GPIO2") (unit 1) (value "RCU-0C") (footprint "RCU-0C:TP+195X110")
     )
+    (path "/4e3b3fe9-0bb8-4770-9e42-7c6ac66f14a3"
+      (reference "H1") (unit 1) (value "MountingHole_Pad") (footprint "MountingHole:MountingHole_3mm")
+    )
+    (path "/684dd7fc-eab4-4bab-96df-b884c79be082"
+      (reference "H2") (unit 1) (value "MountingHole_Pad") (footprint "MountingHole:MountingHole_3mm")
+    )
+    (path "/3cf646a1-f4ce-429d-97ec-f3726b609f92"
+      (reference "H3") (unit 1) (value "MountingHole_Pad") (footprint "MountingHole:MountingHole_3mm")
+    )
+    (path "/ac59f9d0-b2a2-42b3-a2a3-48aa25290f67"
+      (reference "H4") (unit 1) (value "MountingHole_Pad") (footprint "MountingHole:MountingHole_3mm")
+    )
     (path "/9f790417-54e9-48d5-9bdd-b1b4bb15daef"

Commit message: added holes
Parts:
- removed H3: MountingHole_Pad, MountingHole:MountingHole_3mm, symbol Mechanical:MountingHole_Pad
- removed R1: 200k, Resistor_SMD:R_0603_1608Metric, symbol Device:R_Small_US
- removed R2: 270k, Resistor_SMD:R_0603_1608Metric, symbol Device:R_Small_US
- H1, H2, H4: footprint MountingHole:MountingHole_3mm -> MountingHole:MountingHole_3mm_Pad
Connections:
- net GND: no longer IC1.A1 (GND_1), IC1.A2 (GND_2), IC1.A3 (GND_3), IC1.A7 (TST2), IC1.B1 (GND_4), IC1.B2 (GND_5), IC1.B3 (GND_6), IC1.B7 (OVLO), IC1.C1 (GND_7), IC1.C2 (GND_8), IC1.C3 (GND_9), IC1.C4 (GND_10), IC1.C5 (GND_11), IC1.D1 (GND_12), IC1.D2 (GND_13), IC1.D3 (GND_14), IC1.D4 (GND_15), IC1.D5 (GND_16), IC1.D7 (GND_17), IC1.E1 (GND_18), IC1.E2 (GND_19), IC1.E3 (GND_20), IC1.E4 (GND_21), IC1.E5 (GND_22), IC1.F1 (GND_23), IC1.F2 (GND_24), IC1.G1 (GND_25), IC1.G2 (GND_26), IC1.G6 (SYNC), R3.2
- net VBUS_Rdy: now reaches C6.1, FB1.2, FB2.2, IC1.A4 (VIN_1), IC1.A5 (VIN_2), IC1.A6 (SVIN), IC1.B4 (VIN_3), IC1.B5 (VIN_4)
- net VBUS_Rdy: now also IC1.B6 (EN/UVLO)
- new net: IC1.A1 (GND_1), IC1.A2 (GND_2), IC1.A3 (GND_3), IC1.A7 (TST2), IC1.B1 (GND_4), IC1.B2 (GND_5), IC1.B3 (GND_6), IC1.B7 (OVLO), IC1.C1 (GND_7), IC1.C2 (GND_8), IC1.C3 (GND_9), IC1.C4 (GND_10), IC1.C5 (GND_11), IC1.D1 (GND_12), IC1.D2 (GND_13), IC1.D3 (GND_14), IC1.D4 (GND_15), IC1.D5 (GND_16), IC1.D7 (GND_17), IC1.E1 (GND_18), IC1.E2 (GND_19), IC1.E3 (GND_20), IC1.E4 (GND_21), IC1.E5 (GND_22), IC1.F1 (GND_23), IC1.F2 (GND_24), IC1.G1 (GND_25), IC1.G2 (GND_26), IC1.G6 (SYNC), R3.2
Other:
- moved on the sheet: H4

Commit message: layout done!
Connections:
- net GND: now also IC1.A1 (GND_1), IC1.A2 (GND_2), IC1.A3 (GND_3), IC1.A7 (TST2), IC1.B1 (GND_4), IC1.B2 (GND_5), IC1.B3 (GND_6), IC1.B7 (OVLO), IC1.C1 (GND_7), IC1.C2 (GND_8), IC1.C3 (GND_9), IC1.C4 (GND_10), IC1.C5 (GND_11), IC1.D1 (GND_12), IC1.D2 (GND_13), IC1.D3 (GND_14), IC1.D4 (GND_15), IC1.D5 (GND_16), IC1.D7 (GND_17), IC1.E1 (GND_18), IC1.E2 (GND_19), IC1.E3 (GND_20), IC1.E4 (GND_21), IC1.E5 (GND_22), IC1.F1 (GND_23), IC1.F2 (GND_24), IC1.G1 (GND_25), IC1.G2 (GND_26), IC1.G6 (SYNC), R3.2
Changed lines of the file:
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@@
+    (pin "1")
+  )
+  (symbol (lib_id "power:GND") (at 115.57 203.2 0) (unit 1)
+    (in_bom yes) (on_board yes) (fields_autoplaced)
+    (property "Reference" "#PWR0102" (id 0) (at 115.57 209.55 0)
+      (effects (font (size 1.27 1.27)) hide)
+    )
+    (property "Value" "GND" (id 1) (at 115.57 207.645 0))
+    (property "Footprint" "" (id 2) (at 115.57 203.2 0)
+      (effects (font (size 1.27 1.27)) hide)
+    )
+    (property "Datasheet" "" (id 3) (at 115.57 203.2 0)
+      (effects (font (size 1.27 1.27)) hide)
+    )
     (pin "1")
   )
@@
       (reference "#PWR0101") (unit 1) (value "GND") (footprint "")
     )
+    (path "/bf1f8108-d577-4329-93ff-c6541d59441c"
+      (reference "#PWR0102") (unit 1) (value "GND") (footprint "")
+    )
     (path "/5fa9c18e-a21f-4331-abe2-b895eed2ac96"
